File: Robot sumo/PCB/Sumo/Sumo.kicad_pcb (KiCad board)
At the start: 2 copper layers, 65.1 x 44 mm, 33 parts, among them J1 Screw_Terminal_01x01, J2 Screw_Terminal_01x01, J3 Screw_Terminal_01x01, J4 Bat, J5 Screw_Terminal_01x01, M1 M1, M2 M2, U1 MT3608, U2 L293D

Commit message: Added BOM
Parts:
- renumbered EN34 to EN, EN12 to EN, J4 to J3, J3 to J4
Changed lines of the file:
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@@
   (footprint "footprint:WE-PDA" (layer "F.Cu")
     (at 134.874 86.54 180)
+    (property "Mouser Part Number" "710-784771100")
     (property "Sheetfile" "Sumo.kicad_sch")
     (property "Sheetname" "")
@@
     (property "ki_keywords" "inductor choke coil reactor magnetic")
     (attr smd)
-    (fp_text reference "L1" (at 3.302 7.292 unlocked) (layer "F.SilkS")
-        (effects (font (size 1 1) (thickness 0.15)))
-    )
-    (fp_text value "10u" (at 14.126 -0.04 90 unlocked) (layer "F.Fab")
+    (fp_text reference "L1" (at 4.174 7.54 unlocked) (layer "F.SilkS")
+        (effects (font (size 1 1) (thickness 0.15)))
+    )
+    (fp_text value "10u" (at 7.5 0 90 unlocked) (layer "F.Fab")
         (effects (font (size 1 1) (thickness 0.15)))
     )
@@
     (descr "16-lead though-hole mounted DIP package, row spacing 7.62 mm (300 mils)")
     (tags "THT DIP DIL PDIP 2.54mm 7.62mm 300mil")
+    (property "Mouser Part Number" "595-L293DNE")
     (property "Sheetfile" "Sumo.kicad_sch")
     (property "Sheetname" "")
@@
     (descr "Fuse SMD 0805 (2012 Metric), square (rectangular) end terminal, IPC_7351 nominal with elongated pad for handsoldering. (Body size source: https://docs.google.com/spreadsheets/d/1BsfQQcO9C6DZCsRaXUlFlo91Tg2WpOkGARC1WS5S8t0/edit?usp=sharing), generated with kicad-footprint-generator")
     (tags "fuse handsolder")
+    (property "Mouser Part Number" "594-MFU0805FF05000P1")
     (property "Sheetfile" "Sumo.kicad_sch")
     (property "Sheetname" "")
@@
     (descr "Diode SMC (DO-214AB)")
     (tags "Diode SMC (DO-214AB)")
+    (property "Mouser Part Number" "78-VS-MBRS340-M39AT")
     (property "Sheetfile" "Sumo.kicad_sch")
     (property "Sheetname" "")
@@
     (descr "SOT, 6 Pin (https://www.jedec.org/sites/default/files/docs/Mo-178c.PDF variant AB), generated with kicad-footprint-generator ipc_gullwing_generator.py")
     (tags "SOT TO_SOT_SMD")
+    (property "Mouser Part Number" "909-SMDICMT3608")
     (property "Sheetfile" "Sumo.kicad_sch")
     (property "Sheetname" "")
@@
     (property "ki_keywords" "test point tp")
     (attr exclude_from_pos_files)
-    (fp_text reference "EN34" (at 0 -1.648) (layer "F.SilkS")
+    (fp_text reference "EN" (at 0 -1.648) (layer "F.SilkS")
         (effects (font (size 1 1) (thickness 0.15)))
     )
@@
     (property "ki_keywords" "screw terminal")
     (attr exclude_from_pos_files)
-    (fp_text reference "J3" (at 0 -3.8) (layer "F.SilkS") hide
+    (fp_text reference "J4" (at 0 -3.8) (layer "F.SilkS") hide
         (effects (font (size 1 1) (thickness 0.15)))
     )
@@
     (property "ki_keywords" "connector")
     (attr through_hole)
-    (fp_text reference "J4" (at 1.1 -2.006 90) (layer "F.SilkS")
+    (fp_text reference "J3" (at 1.1 -2.006 90) (layer "F.SilkS")
         (effects (font (size 1 1) (thickness 0.15)))
     )
@@
     (property "ki_keywords" "test point tp")
     (attr exclude_from_pos_files)
-    (fp_text reference "EN12" (at 0 -1.648) (layer "F.SilkS")
+    (fp_text reference "EN" (at 0 -1.648) (layer "F.SilkS")
         (effects (font (size 1 1) (thickness 0.15)))
     )
@@
     (descr "Diode SMC (DO-214AB)")
     (tags "Diode SMC (DO-214AB)")
-    (property "Sheetfile" "Sumo.kicad_sch")
-    (property "Sheetname" "")
+    (property "Mouser Part Number" "78-VS-MBRS340-M39AT")
+    (property "Sheetfile" "Sumo.kicad_sch")
+    (property "Sheetname" "")
