File: Robot sumo/PCB/Sumo/Sumo.kicad_sch (KiCad schematic)
At the start: 31 parts, among them J1 Screw_Terminal_01x01, J2 Screw_Terminal_01x01, J3 Bat, J4 Screw_Terminal_01x01, J5 Screw_Terminal_01x01, M1 M1, M2 M2, U1 MT3608, U2 L293D

Commit message: Added BOM
Parts:
- D1, D2: Mouser Part Number (none) -> 78-VS-MBRS340-M39AT
- F1: Mouser Part Number (none) -> 594-MFU0805FF05000P1
- L1: Mouser Part Number (none) -> 710-784771100
- U1: Mouser Part Number (none) -> 909-SMDICMT3608
- U2: Mouser Part Number (none) -> 595-L293DNE
- renumbered 1A to 1A1, 2A to 2A1, 3A to 3A1, 4A to 4A1, BT to BT1, EN12 to EN1, EN34 to EN2, RX to RX1, TX to TX1
Changed lines of the file:
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@@
       (effects (font (size 1.27 1.27)) hide)
     )
-    (property "Datasheet" "~" (at 136.525 41.275 0)
+    (property "Datasheet" "https://www.vishay.com/docs/95748/vs-mbrs340m3.pdf" (at 136.525 41.275 0)
+      (effects (font (size 1.27 1.27)) hide)
+    )
+    (property "Mouser Part Number" "78-VS-MBRS340-M39AT" (at 136.525 41.275 0)
       (effects (font (size 1.27 1.27)) hide)
     )
@@
       (effects (font (size 1.27 1.27)) hide)
     )
-    (property "Datasheet" "~" (at 66.548 46.609 0)
+    (property "Datasheet" "https://www.vishay.com/docs/95748/vs-mbrs340m3.pdf" (at 66.548 46.609 0)
+      (effects (font (size 1.27 1.27)) hide)
+    )
+    (property "Mouser Part Number" "78-VS-MBRS340-M39AT" (at 66.548 46.609 90)
       (effects (font (size 1.27 1.27)) hide)
     )
@@
   (symbol (lib_id "Connector:TestPoint") (at 65.405 107.95 0) (unit 1)
     (in_bom yes) (on_board yes) (dnp no) (fields_autoplaced)
-    (property "Reference" "RX" (at 66.802 104.0043 0)
+    (property "Reference" "RX1" (at 66.802 104.0043 0)
       (effects (font (size 1.27 1.27)) (justify left))
     )
@@
       (project "Sumo"
         (path "/e63e39d7-6ac0-4ffd-8aa3-1841a4541b55"
-          (reference "RX") (unit 1)
+          (reference "RX1") (unit 1)
         )
       )
@@
   (symbol (lib_id "Connector:TestPoint") (at 196.977 117.475 0) (unit 1)
     (in_bom yes) (on_board yes) (dnp no) (fields_autoplaced)
-    (property "Reference" "2A" (at 198.374 113.5293 0)
+    (property "Reference" "2A1" (at 198.374 113.5293 0)
       (effects (font (size 1.27 1.27)) (justify left))
     )
@@
       (project "Sumo"
         (path "/e63e39d7-6ac0-4ffd-8aa3-1841a4541b55"
-          (reference "2A") (unit 1)
+          (reference "2A1") (unit 1)
         )
       )
@@
   (symbol (lib_id "Connector:TestPoint") (at 196.977 122.555 0) (unit 1)
     (in_bom yes) (on_board yes) (dnp no) (fields_autoplaced)
-    (property "Reference" "EN12" (at 198.374 118.6093 0)
+    (property "Reference" "EN1" (at 198.374 118.6093 0)
       (effects (font (size 1.27 1.27)) (justify left))
     )
@@
       (project "Sumo"
         (path "/e63e39d7-6ac0-4ffd-8aa3-1841a4541b55"
-          (reference "EN12") (unit 1)
+          (reference "EN1") (unit 1)
         )
       )
@@
     )
     (property "Datasheet" "http://www.ti.com/lit/ds/symlink/l293.pdf" (at 213.36 109.855 0)
+      (effects (font (size 1.27 1.27)) hide)
+    )
+    (property "Mouser Part Number" "595-L293DNE" (at 220.98 127.635 0)
       (effects (font (size 1.27 1.27)) hide)
     )
@@
       (effects (font (size 1.27 1.27)) hide)
     )
-    (property "Datasheet" "~" (at 57.15 41.275 0)
+    (property "Datasheet" "https://www.vishay.com/docs/28747/mfuserie.pdf" (at 57.15 41.275 0)
+      (effects (font (size 1.27 1.27)) hide)
+    )
+    (property "Mouser Part Number" "594-MFU0805FF05000P1" (at 57.15 41.275 90)
       (effects (font (size 1.27 1.27)) hide)
     )
@@
     )
     (property "Datasheet" "https://www.olimex.com/Products/Breadboarding/BB-PWR-3608/resources/MT3608.pdf" (at 114.3 32.385 0)
+      (effects (font (size 1.27 1.27)) hide)
+    )
+    (property "Mouser Part Number" "909-SMDICMT3608" (at 120.65 43.815 0)
       (effects (font (size 1.27 1.27)) hide)
     )
@@
       (effects (font (size 1.27 1.27)) hide)
     )
-    (property "Datasheet" "~" (at 120.65 30.48 0)
+    (property "Datasheet" "https://www.we-online.com/components/products/datasheet/784771100.pdf" (at 120.65 30.48 0)
+      (effects (font (size 1.27 1.27)) hide)
+    )
+    (property "Mouser Part Number" "710-784771100" (at 120.65 30.48 90)
       (effects (font (size 1.27 1.27)) hide)
     )
@@
   (symbol (lib_id "Connector:TestPoint") (at 196.977 112.395 0) (unit 1)
     (in_bom yes) (on_board yes) (dnp no) (fields_autoplaced)
-    (property "Reference" "1A" (at 198.374 108.4493 0)
+    (property "Reference" "1A1" (at 198.374 108.4493 0)
       (effects (font (size 1.27 1.27)) (justify left))
     )
@@
       (project "Sumo"
         (path "/e63e39d7-6ac0-4ffd-8aa3-1841a4541b55"
-          (reference "1A") (unit 1)
+          (reference "1A1") (unit 1)
         )
       )
@@
   (symbol (lib_id "Connector:TestPoint") (at 196.977 127.635 0) (unit 1)
     (in_bom yes) (on_board yes) (dnp no) (fields_autoplaced)
-    (property "Reference" "3A" (at 198.374 123.6893 0)
+    (property "Reference" "3A1" (at 198.374 123.6893 0)
       (effects (font (size 1.27 1.27)) (justify left))
     )
@@
       (project "Sumo"
         (path "/e63e39d7-6ac0-4ffd-8aa3-1841a4541b55"
-          (reference "3A") (unit 1)
+          (reference "3A1") (unit 1)
         )
       )
@@
   (symbol (lib_id "Connector:TestPoint") (at 196.977 137.795 0) (unit 1)
     (in_bom yes) (on_board yes) (dnp no) (fields_autoplaced)
-    (property "Reference" "EN34" (at 198.374 133.8493 0)
+    (property "Reference" "EN2" (at 198.374 133.8493 0)
       (effects (font (size 1.27 1.27)) (justify left))
     )
@@
       (project "Sumo"
         (path "/e63e39d7-6ac0-4ffd-8aa3-1841a4541b55"
-          (reference "EN34") (unit 1)
+          (reference "EN2") (unit 1)
         )
       )
@@
   (symbol (lib_id "Connector:TestPoint") (at 196.977 132.715 0) (unit 1)
     (in_bom yes) (on_board yes) (dnp no) (fields_autoplaced)
-    (property "Reference" "4A" (at 198.374 128.7693 0)
+    (property "Reference" "4A1" (at 198.374 128.7693 0)
       (effects (font (size 1.27 1.27)) (justify left))
     )
@@
       (project "Sumo"
         (path "/e63e39d7-6ac0-4ffd-8aa3-1841a4541b55"
-          (reference "4A") (unit 1)
+          (reference "4A1") (unit 1)
         )
       )
@@
   (symbol (lib_id "Connector:TestPoint") (at 59.69 111.76 0) (unit 1)
     (in_bom yes) (on_board yes) (dnp no) (fields_autoplaced)
-    (property "Reference" "TX" (at 61.087 107.8143 0)
+    (property "Reference" "TX1" (at 61.087 107.8143 0)
       (effects (font (size 1.27 1.27)) (justify left))
     )
@@
       (project "Sumo"
         (path "/e63e39d7-6ac0-4ffd-8aa3-1841a4541b55"
-          (reference "TX") (unit 1)
+          (reference "TX1") (unit 1)
         )
       )
@@
   (symbol (lib_id "Connector:Conn_01x06_Female") (at 53.34 116.205 0) (mirror y) (unit 1)
     (in_bom yes) (on_board yes) (dnp no) (fields_autoplaced)
-    (property "Reference" "BT" (at 53.975 109.5789 0)
+    (property "Reference" "BT1" (at 53.975 109.5789 0)
       (effects (font (size 1.27 1.27)))
     )
@@
       (project "Sumo"
         (path "/e63e39d7-6ac0-4ffd-8aa3-1841a4541b55"
-          (reference "BT") (unit 1)
-        )
-      )
+          (reference "BT1") (unit 1)
+        )
+      )
